File: Hardware/piDrummer.kicad_pcb (KiCad board)
At the start: 2 copper layers, 96 x 76 mm, 21 parts, among them P1 Trigs_1, P2 Trigs_2, P3 Trigs_3, P4 ROT_ENCODER, P5 ILI9341, P6 Trigs_4, P7 CONN_02X20, Q1 FDD8447L, SW1 Switch_POWER, SW2 Switch_ESCAPE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

Commit message: Added gerber output for hardware
Parts:
- renumbered REF** to ?
Routing:
- net /SW_ESC: track 71.4 -> 57.4 mm
- net /SW_PLAY: track 60.3 -> 50.1 mm
Changed lines of the file:
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@@
   (general
     (links 72)
-    (no_connects 20)
-    (area 15.924999 13.924999 112.075001 90.075001)
+    (no_connects 0)
+    (area 15.924999 12.375 112.075001 91.475)
     (thickness 1.6)
     (drawings 4)
-    (tracks 343)
+    (tracks 341)
     (zones 0)
     (modules 21)
@@
   )
   (setup
-    (last_trace_width 1)
+    (last_trace_width 0.25)
+    (user_trace_width 0.2)
     (user_trace_width 0.5)
     (user_trace_width 1)
@@
     (visible_elements FFFFFF7F)
     (pcbplotparams
-      (layerselection 0x00030_80000001)
-      (usegerberextensions false)
+      (layerselection 0x010f0_80000001)
+      (usegerberextensions true)
       (excludeedgelayer true)
       (linewidth 0.100000)
@@
       (outputformat 1)
       (mirror false)
-      (drillshape 1)
+      (drillshape 0)
       (scaleselection 1)
-      (outputdirectory ""))
+      (outputdirectory OUTPUT_GERBER/))
   )
   (net 0 "")
@@
     (descr "Mounting Hole 4.5mm, no annular")
     (tags "mounting hole 4.5mm no annular")
-    (fp_text reference REF** (at 0 -5.5) (layer F.SilkS)
+    (fp_text reference "" (at -6.035 -3.125) (layer F.SilkS)
       (effects (font (size 1 1) (thickness 0.15)))
     )
@@
     (descr "Mounting Hole 4.5mm, no annular")
     (tags "mounting hole 4.5mm no annular")
-    (fp_text reference REF** (at 0 -5.5) (layer F.SilkS)
+    (fp_text reference "" (at 0 -5.5) (layer F.SilkS)
       (effects (font (size 1 1) (thickness 0.15)))
     )
@@
     (descr "Mounting Hole 4.5mm, no annular")
     (tags "mounting hole 4.5mm no annular")
-    (fp_text reference REF** (at 0 -5.5) (layer F.SilkS)
+    (fp_text reference "" (at 0 -5.5) (layer F.SilkS)
       (effects (font (size 1 1) (thickness 0.15)))
     )
@@
     (descr "Through hole pin header")
     (tags "pin header")
-    (fp_text reference P6 (at 0 -5.1 90) (layer F.SilkS)
+    (fp_text reference P6 (at 1.27 -2.54 90) (layer F.SilkS)
       (effects (font (size 1 1) (thickness 0.15)))
     )
@@
     (fp_arc (start 1.311 0.034) (end 3.051 0.994) (angle 110) (layer F.SilkS) (width 0.15))
     (fp_arc (start 1.301 0.034) (end 2.335 1.094) (angle 87.5) (layer F.SilkS) (width 0.15))
-    (fp_text user K (at -1.69 1.74) (layer F.SilkS)
+    (fp_text user K (at -1.905 0) (layer F.SilkS)
       (effects (font (size 1 1) (thickness 0.15)))
     )
@@
     (descr "Resitance 4 pas")
     (tags R)
-    (fp_text reference R1 (at 0 0 180) (layer F.SilkS)
-      (effects (font (size 1 1) (thickness 0.15)))
-    )
-    (fp_text value 100 (at 0 0 180) (layer F.Fab)
+    (fp_text reference R1 (at 2.54 0 180) (layer F.SilkS)
+      (effects (font (size 1 1) (thickness 0.15)))
+    )
+    (fp_text value 100 (at -2.54 0 180) (layer F.Fab)
       (effects (font (size 1 1) (thickness 0.15)))
     )
@@
     (descr "Resitance 4 pas")
     (tags R)
-    (fp_text reference R2 (at 0 0 180) (layer F.SilkS)
-      (effects (font (size 1 1) (thickness 0.15)))
-    )
-    (fp_text value 330 (at 0 0 180) (layer F.Fab)
+    (fp_text reference R2 (at 2.54 0 180) (layer F.SilkS)
+      (effects (font (size 1 1) (thickness 0.15)))
+    )
+    (fp_text value 330 (at -2.54 0 180) (layer F.Fab)
       (effects (font (size 1 1) (thickness 0.15)))
     )
@@
     (descr "Resitance 4 pas")
     (tags R)
-    (fp_text reference R3 (at 0 0 270) (layer F.SilkS)
-      (effects (font (size 1 1) (thickness 0.15)))
-    )
-    (fp_text value 2K2 (at 0 0 270) (layer F.Fab)
+    (fp_text reference R3 (at 2.54 0 270) (layer F.SilkS)
+      (effects (font (size 1 1) (thickness 0.15)))
+    )
+    (fp_text value 2K2 (at -2.54 0 270) (layer F.Fab)
       (effects (font (size 1 1) (thickness 0.15)))
     )
@@
     (descr "Resitance 4 pas")
     (tags R)
-    (fp_text reference R4 (at 0 0 270) (layer F.SilkS)
-      (effects (font (size 1 1) (thickness 0.15)))
-    )
-    (fp_text value 3K3 (at 0 0 270) (layer F.Fab)
+    (fp_text reference R4 (at 2.54 0 270) (layer F.SilkS)
+      (effects (font (size 1 1) (thickness 0.15)))
+    )
+    (fp_text value 3K3 (at -2.54 0 270) (layer F.Fab)
       (effects (font (size 1 1) (thickness 0.15)))
     )
@@
     (descr "30 pins DIL package, elliptical pads, width 600mil (arduino mini)")
     (tags "DIL arduino mini")
-    (fp_text reference U1 (at -13.97 -3.81) (layer F.SilkS)
+    (fp_text reference U1 (at -1.27 0) (layer F.SilkS)
       (effects (font (size 1.778 1.778) (thickness 0.3048)))
     )
@@
     (tags "D-Pak TO252AA Diode")
     (attr smd)
-    (fp_text reference Q1 (at 0 -7.5 90) (layer F.SilkS)
-      (effects (font (size 1 1) (thickness 0.15)))
-    )
-    (fp_text value FDD8447L (at 4.445 -1.905 360) (layer F.Fab)
+    (fp_text reference Q1 (at 0 -8.255 90) (layer F.SilkS)
+      (effects (font (size 1 1) (thickness 0.15)))
+    )
+    (fp_text value FDD8447L (at 0 -6.35 90) (layer F.Fab)
       (effects (font (size 1 1) (thickness 0.15)))
     )
@@
     (descr "Through hole pin header")
     (tags "pin header")
-    (fp_text reference P1 (at 0 -5.1 90) (layer F.SilkS)
+    (fp_text reference P1 (at 1.27 -2.54 90) (layer F.SilkS)
       (effects (font (size 1 1) (thickness 0.15)))
     )
@@
     (descr "Through hole pin header")
     (tags "pin header")
-    (fp_text reference P2 (at 0 -5.1 90) (layer F.SilkS)
+    (fp_text reference P2 (at 1.27 -2.54 90) (layer F.SilkS)
       (effects (font (size 1 1) (thickness 0.15)))
     )
@@
     (descr "Through hole pin header")
     (tags "pin header")
-    (fp_text reference P3 (at 0 -5.1 90) (layer F.SilkS)
+    (fp_text reference P3 (at 1.27 -2.54 90) (layer F.SilkS)
       (effects (font (size 1 1) (thickness 0.15)))
     )
@@
     (descr "Through hole pin header")
     (tags "pin header")
-    (fp_text reference P4 (at 0 -5.1 270) (layer F.SilkS)
+    (fp_text reference P4 (at 1.905 -0.635 360) (layer F.SilkS)
       (effects (font (size 1 1) (thickness 0.15)))
     )
@@
     (descr "Mounting Hole 4.5mm, no annular")
     (tags "mounting hole 4.5mm no annular")
-    (fp_text reference REF** (at 0 -5.5) (layer F.SilkS)
+    (fp_text reference "" (at 0 -5.5) (layer F.SilkS)
       (effects (font (size 1 1) (thickness 0.15)))
     )
@@
   (segment (start 83.82 34.925) (end 83.82 23.495) (width 0.5) (layer B.Cu) (net 20))
   (segment (start 62.865 36.83) (end 81.915 36.83) (width 0.5) (layer B.Cu) (net 20))
-  (segment (start 83.185 22.86) (end 58.42 22.86) (width 0.5) (layer B.Cu) (net 20) (status 800000))
+  (segment (start 83.185 22.86) (end 58.42 22.86) (width 0.5) (layer B.Cu) (net 20))
   (segment (start 83.82 23.495) (end 83.185 22.86) (width 0.5) (layer B.Cu) (net 20))
   (segment (start 57.15 35.56) (end 57.15 34.29) (width 0.5) (layer B.Cu) (net 20))
@@
   (segment (start 86.36 20.32) (end 86.36 36.83) (width 1) (layer B.Cu) (net 24))
   (segment (start 86.36 36.83) (end 80.01 43.18) (width 1) (layer B.Cu) (net 24))
-  (segment (start 64.77 43.18) (end 80.01 43.18) (width 1) (layer B.Cu) (net 24) (status 400000))
+  (segment (start 64.77 43.18) (end 80.01 43.18) (width 1) (layer B.Cu) (net 24))
   (segment (start 84.455 18.415) (end 62.23 18.415) (width 1) (layer B.Cu) (net 24))
   (segment (start 86.36 20.32) (end 84.455 18.415) (width 1) (layer B.Cu) (net 24))
@@
   (segment (start 58.42 79.375) (end 58.42 80.645) (width 0.25) (layer B.Cu) (net 33))
   (segment (start 57.15 78.105) (end 58.42 79.375) (width 0.25) (layer B.Cu) (net 33))
-  (segment (start 43.18 78.105) (end 57.15 78.105) (width 0.25) (layer B.Cu) (net 33))
   (segment (start 40.64 71.12) (end 40.64 75.565) (width 0.25) (layer B.Cu) (net 33))
   (segment (start 54.61 80.645) (end 49.53 80.645) (width 0.5) (layer B.Cu) (net 34))
@@
   (segment (start 49.53 80.645) (end 47.625 80.645) (width 0.25) (layer B.Cu) (net 34))
   (segment (start 35.56 75.565) (end 35.56 72.39) (width 0.25) (layer B.Cu) (net 34))
-  (segment (start 45.72 82.55) (end 35.56 82.55) (width 0.25) (layer B.Cu) (net 34))
   (segment (start 47.625 80.645) (end 45.72 82.55) (width 0.25) (layer B.Cu) (net 34))
   (zone (net 1) (net_name GND) (layer F.Cu) (hatch edge 0.508)
     (connect_pads (clearance 0.508))
     (min_thickness 0.254)
-    (fill (arc_segments 16) (thermal_gap 0.508) (thermal_bridge_width 0.508))
+    (fill yes (arc_segments 16) (thermal_gap 0.508) (thermal_bridge_width 0.508))
     (polygon
       (pts
@@
     (connect_pads (clearance 0.508))
     (min_thickness 0.254)
-    (fill (arc_segments 16) (thermal_gap 0.508) (thermal_bridge_width 0.508))
+    (fill yes (arc_segments 16) (thermal_gap 0.508) (thermal_bridge_width 0.508))
     (polygon
       (pts
