File: Hardware/piDrummer_AD_Board.kicad_pcb (KiCad board)
At the start: 2 copper layers, 72.5 x 80.5 mm, 55 parts, among them P1 CONN_02X04, P2 CONN_02X16, U3 4051, U4 4051

Commit message: Added gerber output for hardware
Parts:
- added ?: , Mounting_Holes:MountingHole_4.5mm, F.Cu at (106.7, 107.3)
- ? (x3): renamed from REF**; value MountingHole_4.5mm -> (none)
- moved ? 6.38 mm to (106.7, 35.6)
Routing:
- net /IN11: track 99.5 -> 47.8 mm
- net /IN7: track 57.1 -> 31.1 mm
- net /MUX1: track 85.1 -> 62.2 mm
- net VCC: track 238.9 -> 223.6 mm
- net /IN3: track 27.5 -> 41.7 mm
- net /IN9: track 72.8 -> 59.4 mm
- net /IN10: track 76.0 -> 67.8 mm
- net /IN1: track 27.6 -> 32.7 mm
- net /IN13: track 42.5 -> 44.5 mm
- net /IN12: track 80.9 -> 81.7 mm
- net /IN5: track 29.4 -> 30.1 mm
Other:
- board size 72.5 x 80.5 mm -> 79 x 80.5 mm
